File: cpu.sch (KiCad schematic (older format))
At the start: 4 parts

Commit message: -
Parts:
- added C? (x8): CAPAPOL, symbol CAPAPOL
- added C? (x2): C, symbol C
- added U? (x2): MC34063A, symbol MC34063A
