File: cpu/cpu.sch (KiCad schematic (older format))
At the start: 16 parts

Commit message: update
Parts:
- C2: renamed from C?; value CAPAPOL -> 470uF 16V
- C5: renamed from C?; value CAPAPOL -> 330uF 16V
- gave numbers to parts that had none: 2
Other:
- moved on the sheet: C1, C2, C4, C5, C?, L1, L2, L3, L4, U?
Changed lines of the file:
@@
 L INDUCTOR L1
 U 1 1 54CBF699
-P 700 900
-F 0 "L1" V 650 900 50  0000 C CNN
-F 1 "INDUCTOR" V 800 900 50  0000 C CNN
-F 2 "" H 700 900 60  0000 C CNN
-F 3 "" H 700 900 60  0000 C CNN
-	1    700  900
+P 12350 550
+F 0 "L1" V 12300 550 50  0000 C CNN
+F 1 "INDUCTOR" V 12450 550 50  0000 C CNN
+F 2 "" H 12350 550 60  0000 C CNN
+F 3 "" H 12350 550 60  0000 C CNN
+	1    12350 550
 	1    0    0    -1
 $EndComp
@@
 L INDUCTOR L2
 U 1 1 54CBF6BA
-P 950 900
-F 0 "L2" V 900 900 50  0000 C CNN
-F 1 "INDUCTOR" V 1050 900 50  0000 C CNN
-F 2 "" H 950 900 60  0000 C CNN
-F 3 "" H 950 900 60  0000 C CNN
-	1    950  900
+P 12600 550
+F 0 "L2" V 12550 550 50  0000 C CNN
+F 1 "INDUCTOR" V 12700 550 50  0000 C CNN
+F 2 "" H 12600 550 60  0000 C CNN
+F 3 "" H 12600 550 60  0000 C CNN
+	1    12600 550
 	1    0    0    -1
 $EndComp
@@
 L INDUCTOR L3
 U 1 1 54CBF8BB
-P 1200 900
-F 0 "L3" V 1150 900 50  0000 C CNN
-F 1 "INDUCTOR" V 1300 900 50  0000 C CNN
-F 2 "" H 1200 900 60  0000 C CNN
-F 3 "" H 1200 900 60  0000 C CNN
-	1    1200 900
+P 12850 550
+F 0 "L3" V 12800 550 50  0000 C CNN
+F 1 "INDUCTOR" V 12950 550 50  0000 C CNN
+F 2 "" H 12850 550 60  0000 C CNN
+F 3 "" H 12850 550 60  0000 C CNN
+	1    12850 550
 	1    0    0    -1
 $EndComp
@@
 L INDUCTOR L4
 U 1 1 54CBF927
-P 1500 900
-F 0 "L4" V 1450 900 50  0000 C CNN
-F 1 "INDUCTOR" V 1600 900 50  0000 C CNN
-F 2 "" H 1500 900 60  0000 C CNN
-F 3 "" H 1500 900 60  0000 C CNN
-	1    1500 900
+P 13150 550
+F 0 "L4" V 13100 550 50  0000 C CNN
+F 1 "INDUCTOR" V 13250 550 50  0000 C CNN
+F 2 "" H 13150 550 60  0000 C CNN
+F 3 "" H 13150 550 60  0000 C CNN
+	1    13150 550
 	1    0    0    -1
 $EndComp
@@
 L MC34063A U?
 U 1 1 54CBFB62
-P 2800 1700
-F 0 "U?" H 2500 2250 60  0000 L CNN
-F 1 "MC34063A" H 2500 1150 60  0000 L CNN
-F 2 "" H 2800 1200 60  0000 C CNN
-F 3 "" H 2800 1200 60  0000 C CNN
-	1    2800 1700
+P 14450 1350
+F 0 "U?" H 14150 1900 60  0000 L CNN
+F 1 "MC34063A" H 14150 800 60  0000 L CNN
+F 2 "" H 14450 850 60  0000 C CNN
+F 3 "" H 14450 850 60  0000 C CNN
+	1    14450 1350
 	1    0    0    -1
 $EndComp
@@
 L MC34063A U?
 U 1 1 54CBFB8F
-P 4550 1700
-F 0 "U?" H 4250 2250 60  0000 L CNN
-F 1 "MC34063A" H 4250 1150 60  0000 L CNN
-F 2 "" H 4550 1200 60  0000 C CNN
-F 3 "" H 4550 1200 60  0000 C CNN
-	1    4550 1700
+P 16200 1350
+F 0 "U?" H 15900 1900 60  0000 L CNN
+F 1 "MC34063A" H 15900 800 60  0000 L CNN
+F 2 "" H 16200 850 60  0000 C CNN
+F 3 "" H 16200 850 60  0000 C CNN
+	1    16200 1350
 	1    0    0    -1
 $EndComp
 $Comp
-L CAPAPOL C?
+L CAPAPOL C2
 U 1 1 54CBFC06
-P 6000 1100
-F 0 "C?" H 6050 1200 50  0000 L CNN
-F 1 "CAPAPOL" H 6050 1000 50  0000 L CNN
-F 2 "" H 6100 950 30  0000 C CNN
-F 3 "" H 6000 1100 300 0000 C CNN
-	1    6000 1100
+P 17650 750
+F 0 "C2" H 17700 850 50  0000 L CNN
+F 1 "470uF 16V" H 17700 650 50  0000 L CNN
+F 2 "" H 17750 600 30  0000 C CNN
+F 3 "" H 17650 750 300 0000 C CNN
+	1    17650 750
 	1    0    0    -1
 $EndComp
 $Comp
-L CAPAPOL C?
+L CAPAPOL C5
 U 1 1 54CBFC51
-P 6350 1100
-F 0 "C?" H 6400 1200 50  0000 L CNN
-F 1 "CAPAPOL" H 6400 1000 50  0000 L CNN
-F 2 "" H 6450 950 30  0000 C CNN
-F 3 "" H 6350 1100 300 0000 C CNN
-	1    6350 1100
+P 18000 750
+F 0 "C5" H 18050 850 50  0000 L CNN
+F 1 "330uF 16V" H 18050 650 50  0000 L CNN
+F 2 "" H 18100 600 30  0000 C CNN
+F 3 "" H 18000 750 300 0000 C CNN
+	1    18000 750
 	1    0    0    -1
 $EndComp
@@
 L CAPAPOL C?
 U 1 1 54CBFD36
-P 6700 1100
-F 0 "C?" H 6750 1200 50  0000 L CNN
-F 1 "CAPAPOL" H 6750 1000 50  0000 L CNN
-F 2 "" H 6800 950 30  0000 C CNN
-F 3 "" H 6700 1100 300 0000 C CNN
-	1    6700 1100
+P 18350 750
+F 0 "C?" H 18400 850 50  0000 L CNN
+F 1 "CAPAPOL" H 18400 650 50  0000 L CNN
+F 2 "" H 18450 600 30  0000 C CNN
+F 3 "" H 18350 750 300 0000 C CNN
+	1    18350 750
 	1    0    0    -1
 $EndComp
@@
 L CAPAPOL C?
 U 1 1 54CBFD3C
-P 7050 1100
-F 0 "C?" H 7100 1200 50  0000 L CNN
-F 1 "CAPAPOL" H 7100 1000 50  0000 L CNN
-F 2 "" H 7150 950 30  0000 C CNN
-F 3 "" H 7050 1100 300 0000 C CNN
-	1    7050 1100
+P 18700 750
+F 0 "C?" H 18750 850 50  0000 L CNN
+F 1 "CAPAPOL" H 18750 650 50  0000 L CNN
+F 2 "" H 18800 600 30  0000 C CNN
+F 3 "" H 18700 750 300 0000 C CNN
+	1    18700 750
 	1    0    0    -1
 $EndComp
@@
 L CAPAPOL C?
 U 1 1 54CBFDCA
-P 6000 1700
-F 0 "C?" H 6050 1800 50  0000 L CNN
-F 1 "CAPAPOL" H 6050 1600 50  0000 L CNN
-F 2 "" H 6100 1550 30  0000 C CNN
-F 3 "" H 6000 1700 300 0000 C CNN
-	1    6000 1700
+P 17650 1350
+F 0 "C?" H 17700 1450 50  0000 L CNN
+F 1 "CAPAPOL" H 17700 1250 50  0000 L CNN
+F 2 "" H 17750 1200 30  0000 C CNN
+F 3 "" H 17650 1350 300 0000 C CNN
+	1    17650 1350
 	1    0    0    -1
 $EndComp
@@
 L CAPAPOL C?
 U 1 1 54CBFDD0
-P 6350 1700
-F 0 "C?" H 6400 1800 50  0000 L CNN
-F 1 "CAPAPOL" H 6400 1600 50  0000 L CNN
-F 2 "" H 6450 1550 30  0000 C CNN
-F 3 "" H 6350 1700 300 0000 C CNN
-	1    6350 1700
+P 18000 1350
+F 0 "C?" H 18050 1450 50  0000 L CNN
+F 1 "CAPAPOL" H 18050 1250 50  0000 L CNN
+F 2 "" H 18100 1200 30  0000 C CNN
+F 3 "" H 18000 1350 300 0000 C CNN
+	1    18000 1350
 	1    0    0    -1
 $EndComp
@@
 L CAPAPOL C?
 U 1 1 54CBFDD6
-P 6700 1700
-F 0 "C?" H 6750 1800 50  0000 L CNN
-F 1 "CAPAPOL" H 6750 1600 50  0000 L CNN
-F 2 "" H 6800 1550 30  0000 C CNN
-F 3 "" H 6700 1700 300 0000 C CNN
-	1    6700 1700
+P 18350 1350
+F 0 "C?" H 18400 1450 50  0000 L CNN
+F 1 "CAPAPOL" H 18400 1250 50  0000 L CNN
+F 2 "" H 18450 1200 30  0000 C CNN
+F 3 "" H 18350 1350 300 0000 C CNN
+	1    18350 1350
 	1    0    0    -1
 $EndComp
@@
 L CAPAPOL C?
 U 1 1 54CBFDDC
-P 7050 1700
-F 0 "C?" H 7100 1800 50  0000 L CNN
-F 1 "CAPAPOL" H 7100 1600 50  0000 L CNN
-F 2 "" H 7150 1550 30  0000 C CNN
-F 3 "" H 7050 1700 300 0000 C CNN
-	1    7050 1700
+P 18700 1350
+F 0 "C?" H 18750 1450 50  0000 L CNN
+F 1 "CAPAPOL" H 18750 1250 50  0000 L CNN
+F 2 "" H 18800 1200 30  0000 C CNN
+F 3 "" H 18700 1350 300 0000 C CNN
+	1    18700 1350
 	1    0    0    -1
 $EndComp
 $Comp
-L C C?
+L C C1
 U 1 1 54CBFE46
-P 7900 1150
-F 0 "C?" H 7950 1250 50  0000 L CNN
-F 1 "C" H 7950 1050 50  0000 L CNN
-F 2 "" H 7938 1000 30  0000 C CNN
-F 3 "" H 7900 1150 60  0000 C CNN
-	1    7900 1150
+P 19550 800
+F 0 "C1" H 19600 900 50  0000 L CNN
+F 1 "C" H 19600 700 50  0000 L CNN
+F 2 "" H 19588 650 30  0000 C CNN
+F 3 "" H 19550 800 60  0000 C CNN
+	1    19550 800
 	1    0    0    -1
 $EndComp
 $Comp
-L C C?
+L C C4
 U 1 1 54CBFEB1
-P 8250 1150
-F 0 "C?" H 8300 1250 50  0000 L CNN
-F 1 "C" H 8300 1050 50  0000 L CNN
-F 2 "" H 8288 1000 30  0000 C CNN
-F 3 "" H 8250 1150 60  0000 C CNN
-	1    8250 1150
+P 19900 800
+F 0 "C4" H 19950 900 50  0000 L CNN
+F 1 "C" H 19950 700 50  0000 L CNN
+F 2 "" H 19938 650 30  0000 C CNN
+F 3 "" H 19900 800 60  0000 C CNN
+	1    19900 800
 	1    0    0    -1
 $EndComp
+$Sheet
+S 11900 -300 19050 10400
+U 54D7BF2C
+F0 "Sheet_psu" 60
+F1 "psu.sch" 60
+$EndSheet
 $EndSCHEMATC
